File: wi-min.sch (KiCad schematic (older format))
At the start: 6 parts, among them CON1 AVR-ISP-6, IC1 ATMEGA8A-P, P1 BAT_3V, P2 NRF24_CONN_5X2, P3 CONN_4

Commit message: post v2
Parts:
- removed C1: SERIAL_TTL_3.5MM, ~, symbol SERIAL_TTL_3.5MM
- removed P1: BAT_3V, symbol CONN_2
- added C2, C3: C, ~, symbol C
- added D1: LED, ~, symbol LED
- added JP1: JUMPER, ~, symbol JUMPER
- added P1: BATTERY, ~, symbol BATTERY
- added P4: 3F07, 3F07, symbol 3F07
- added R1, R2: R, ~, symbol R
- added SW1: SPST, ~, symbol SPST
- added X1: CRYSTAL_W_GND, ~, symbol CRYSTAL_W_GND
Connections:
- net labels added: CE, CSN, DBG_LED, IRQ, TOSC1, TOSC2
- net labels removed: INT0
- wire segments 32 -> 24
- no-connect marks 0 -> 2
Other:
- note added: "What was the point of this jumper?"
- moved on the sheet: CON1

Commit message: v3 sent for fabrication
Parts:
- removed IC1: ATMEGA8A-P, DIL28, symbol ATMEGA8A-P
- removed JP1: JUMPER, ~, symbol JUMPER
- added C1, C4: C, ~, symbol C
- added D2: LED, ~, symbol LED
- added IC1: ATMEGA8-AI, TQFP32, symbol ATMEGA8-AI
- added R3: R, ~, symbol R
- added R4: 150R, ~, symbol R
- added SW2: SPST, ~, symbol SPST
- R2: value R -> 150R
Connections:
- net CE: now also IC1.23 ((ADC0)PC0)
- net CSN: now also IC1.24 ((ADC1)PC1)
- net GND: now also C1.2, C4.2, D2.2 (K), IC1.21 (AGND), IC1.3 (GND), IC1.5 (GND), SW2.1
- net IRQ: now also IC1.32 ((INT0)PD2)
- net MISO: now also IC1.16 ((MISO)PB4)
- net MOSI: now also IC1.15 ((MOSI/OC2)PB3)
- net RST: now also C4.1, IC1.29 (PC6(~RESET~))
- net Rx: now also IC1.31 ((TXD)PD1)
- net SCK: now also IC1.17 ((SCK)PB5)
- net SCL: now also IC1.28 ((ADC5/SCL)PC5)
- net SDA: now also IC1.27 ((ADC4/SDA)PC4)
- net TOSC1: now also IC1.7 (PB6(XTAL1/TOSC1))
- net TOSC2: now also IC1.8 (PB7(XTAL2/TOSC2))
- net Tx: now also IC1.30 ((RXD)PD0)
- net VCC: now also P1.1 (+), IC1.18 (AVCC), IC1.20 (AREF), IC1.4 (VCC), IC1.6 (VCC)
- net DBG_LED renamed LED0
- net LED0: now also IC1.13 ((OC1A)PB1)
- new net: R3.1, SW2.2
- new net: D2.1 (A), R4.2
- new net LED1: IC1.14 ((~SS~/OC1B)PB2), R4.1
- new net USR_BUTTON: C1.1, IC1.12 ((ICP)PB0), R3.2
Other:
- note removed: "What was the point of this jumper?"
- moved on the sheet: P2, P3, P4, R1, SW1
