File: wi-min.kicad_pcb (KiCad board)
At the start: 2 copper layers, 44.4 x 29.2 mm, 6 parts, among them CON1 AVR-ISP-6, IC1 ATMEGA8A-P, P1 BAT_3V, P2 NRF24_CONN_5X2, P3 CONN_4

Commit message: post v2
Parts:
- removed C1: SERIAL_TTL_3.5MM, SIL-3
- added C2: C, SM0603_Capa, F.Cu at (198.1, 119.4)
- added C3: C, SM0603_Capa, F.Cu at (205.7, 105.4)
- added D1: LED, LED-0603, F.Cu at (212.1, 109.2)
- added JP1: JUMPER, SM0402, F.Cu at (198.1, 121.9)
- added P4: 3F07, 3F07, F.Cu at (186.9, 125.7)
- added R1: R, SM0603, F.Cu at (191.8, 109.2)
- added R2: R, SM0603, F.Cu at (207.0, 109.2)
- added SW1: SPST, SW_PUSH_SMALL, F.Cu at (189.2, 102.9)
- added X1: CRYSTAL_W_GND, AB26TRB, F.Cu at (208.3, 113.0)
- CON1: footprint pin_array_3x2 -> atmel-2-AVR-ISP-6
- IC1: footprint DIP-28__300 -> atmel-TQFP32
- P1: value BAT_3V -> BATTERY; footprint SIL-2 -> CR2032_HOLDER_TH; moved to B.Cu
- moved P2 24.7 mm to (200.7, 100.3)
- moved CON1 22.9 mm to (204.5, 120.7)
- moved P1 11.5 mm to (215.8, 109.1)
- moved P3 10.8 mm to (182.9, 108.0), turned to 90 degrees
- moved IC1 4.20 mm to (199.5, 109.8), turned to 90 degrees
Connections:
- net /INT0 renamed /IRQ
- IC1 pad 10: N-000005 -> /TOSC2
- IC1 pad 15: (no net) -> /DBG_LED
- IC1 pad 2: /Rx -> /Tx
- IC1 pad 23: (no net) -> /CE
- IC1 pad 24: (no net) -> /CSN
- IC1 pad 3: /Tx -> /Rx
- IC1 pad 9: N-000009 -> /TOSC1
- P1 pad 1: VCC -> N-0000012
- P2 pad 3: N-000009 -> /CE
- P2 pad 4: N-000005 -> /CSN
Routing:
- net GND: track 22.6 -> 113.5 mm, vias 0 -> 4
- net N-0000012: track 0.00 -> 19.5 mm
- net VCC: track 55.5 -> 74.1 mm
- net /MISO: track 23.3 -> 36.8 mm
- net /RST: track 40.8 -> 30.1 mm
- net /Tx: track 7.40 -> 17.9 mm, vias 1 -> 0
- net N-000001: track 0.00 -> 9.40 mm
- net N-000009: track 9.20 -> 0.00 mm
- net /IRQ: track 27.0 -> 18.4 mm, vias 0 -> 2
- net /CSN: track 0.00 -> 6.99 mm
- net /SCL: track 7.62 -> 14.1 mm, vias 0 -> 1
- net /SDA: track 7.62 -> 12.6 mm
- net N-000005: track 4.86 -> 0.00 mm
- net /CE: track 0.00 -> 4.13 mm
- net /TOSC1: track 0.00 -> 3.97 mm
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Other:
- board size 44.4 x 29.2 mm -> 40.6 x 29.2 mm
- net class Minimal added: clearance 0.1524, trace_width 0.1524, via_dia 0.508, via_drill 0.3302
- rule trace_min: 0.254 -> 0.1524
- rule via_min_drill: 0.508 -> 0.3302
- rule via_min_size: 0.889 -> 0.508
- board text added: "wi-min v2 Cody P Schafer 2013-05-29"
- board text removed: "ISP"
- board text removed: "SCL"
- board text removed: "SDA"
- board text removed: "wi-min v1 Cody P Schafer"

Commit message: v3 sent for fabrication
Parts:
- removed JP1: JUMPER, SM0402
- added C1: C, SM0603_Capa, F.Cu at (209.0, 109.0)
- added C4: C, SM0603_Capa, F.Cu at (192.7, 103.1)
- added D2: LED, LED-0603, F.Cu at (206.2, 105.2)
- added R3: R, SM0603, F.Cu at (209.0, 105.8)
- added R4: 150R, SM0603, F.Cu at (206.2, 107.2)
- added SW2: SPST, SW_PUSH_SMALL, F.Cu at (208.9, 100.3)
- IC1: value ATMEGA8A-P -> ATMEGA8-AI; footprint atmel-TQFP32 -> TQFP32
- P1: footprint CR2032_HOLDER_TH -> CR2032_HOLDER_TH_ON_SIDE
- R2: value R -> 150R
- moved CON1 6.48 mm to (198.1, 121.9), turned to 180 degrees
- moved R1 6.14 mm to (191.0, 103.1)
- moved D1 4.66 mm to (208.0, 111.5)
- moved X1 4.52 mm to (204.7, 115.8), turned to 90 degrees
- moved P1 4.19 mm to (211.6, 109.2)
- moved SW1 4.02 mm to (185.4, 101.6)
- moved P2 3.78 mm to (197.1, 99.1)
- moved P3 3.47 mm to (186.3, 108.5), turned to 0 degrees
- moved C2 3.02 mm to (198.9, 116.5)
- moved C3 2.84 mm to (203.2, 104.1)
- moved IC1 1.48 mm to (198.1, 109.2)
- moved R2 0.76 mm to (206.2, 109.2)
Connections:
- IC1 pad 1: /RST -> (no net)
- IC1 pad 10: /TOSC2 -> (no net)
- IC1 pad 12: (no net) -> /USR_BUTTON
- IC1 pad 13: (no net) -> /LED0
- IC1 pad 14: (no net) -> /LED1
- IC1 pad 15: /DBG_LED -> /MOSI
- IC1 pad 16: (no net) -> /MISO
- IC1 pad 17: /MOSI -> /SCK
- IC1 pad 18: /MISO -> VCC
- IC1 pad 19: /SCK -> (no net)
- IC1 pad 2: /Tx -> (no net)
- IC1 pad 21: VCC -> GND
- IC1 pad 22: GND -> (no net)
- IC1 pad 29: (no net) -> /RST
- IC1 pad 3: /Rx -> GND
- IC1 pad 30: (no net) -> /Tx
- IC1 pad 31: (no net) -> /Rx
- IC1 pad 32: (no net) -> /IRQ
- IC1 pad 4: /IRQ -> VCC
- IC1 pad 5: (no net) -> GND
- IC1 pad 6: (no net) -> VCC
- IC1 pad 7: VCC -> /TOSC1
- IC1 pad 8: GND -> /TOSC2
- IC1 pad 9: /TOSC1 -> (no net)
- P1 pad 1: N-0000012 -> VCC
- R2 pad 1: /DBG_LED -> /LED0
Routing:
- net GND: track 113.5 -> 64.8 mm, vias 4 -> 11
- net /MISO: track 36.8 -> 25.4 mm
- net /USR_BUTTON: track 0.00 -> 10.7 mm
- net N-0000012: track 19.5 -> 8.87 mm
- net VCC: track 74.1 -> 80.7 mm, vias 0 -> 4
- net /MOSI: track 24.6 -> 31.1 mm
- net /RST: track 30.1 -> 24.2 mm, vias 1 -> 2
- net N-0000030: track 9.40 -> 5.13 mm
- net /SDA: track 12.6 -> 9.24 mm
- net /TOSC2: track 3.25 -> 6.36 mm
- net /DBG_LED: track 3.04 -> 0.00 mm
- net /LED1: track 0.00 -> 2.95 mm
- net /LED0: track 0.00 -> 2.74 mm
- net /SCL: track 14.1 -> 12.0 mm, vias 1 -> 0
- net N-0000014: track 0.00 -> 2.04 mm
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Other:
- board size 40.6 x 29.2 mm -> 34 x 29.2 mm
- board text added: "wi-min v3 Cody P Schafer 2013-06-20"
- board text removed: "wi-min v2 Cody P Schafer 2013-05-29"

Commit message: post v3 changes
Routing:
- net GND: track 64.8 -> 78.1 mm, vias 11 -> 14
- net /IRQ: track 18.3 -> 26.3 mm
Other:
- board text added: "wi-min v4 Cody P Schafer 2013-06-25"
- board text removed: "wi-min v3 Cody P Schafer 2013-06-20"
Changed lines of the file:
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@@
     (area 180.289999 96.469999 214.426001 125.780001)
     (thickness 1.6)
-    (drawings 29)
-    (tracks 204)
+    (drawings 33)
+    (tracks 216)
     (zones 0)
     (modules 19)
@@
   (module AB26TRB (layer F.Cu)
     (at 204.724 115.824 90)
-    (fp_text reference X1 (at -5.334 -3.048 90) (layer F.SilkS)
+    (fp_text reference X1 (at -1.524 2.667 90) (layer F.SilkS)
       (effects (font (size 1.524 1.524) (thickness 0.3048)))
     )
@@
     )
   )
+  (gr_arc (start 201.676 119.634) (end 201.676 118.618) (angle 90) (layer F.SilkS) (width 0.2))
+  (gr_arc (start 202.057 120.65) (end 202.819 119.888) (angle 90) (layer F.SilkS) (width 0.2))
+  (gr_arc (start 200.66 119.253) (end 199.898 118.491) (angle 90) (layer F.SilkS) (width 0.2))
+  (gr_circle (center 200.66 120.65) (end 202.057 121.031) (layer F.SilkS) (width 0.2))
   (gr_line (start 214.376 96.52) (end 180.34 96.52) (angle 90) (layer Edge.Cuts) (width 0.1))
   (gr_line (start 180.34 125.73) (end 214.376 125.73) (angle 90) (layer Edge.Cuts) (width 0.1))
@@
   (gr_line (start 214.376 125.73) (end 214.376 96.52) (angle 90) (layer Edge.Cuts) (width 0.1))
   (gr_line (start 180.34 96.52) (end 180.34 125.73) (angle 90) (layer Edge.Cuts) (width 0.1))
-  (gr_text "wi-min v3\nCody P Schafer\n2013-06-20" (at 186.309 110.744) (layer F.SilkS)
+  (gr_text "wi-min v4\nCody P Schafer\n2013-06-25" (at 186.309 110.744) (layer F.SilkS)
     (effects (font (size 1.016 1.016) (thickness 0.127)))
   )
@@
   (segment (start 193.294 101.092) (end 193.294 99.06) (width 0.381) (layer F.Cu) (net 2))
   (segment (start 195.3006 103.6066) (end 193.294 101.092) (width 0.381) (layer F.Cu) (net 2))
-  (segment (start 199.644 97.79) (end 199.644 98.171) (width 0.254) (layer B.Cu) (net 3))
-  (segment (start 195.67652 112.04448) (end 193.294 112.04448) (width 0.254) (layer F.Cu) (net 3))
-  (segment (start 198.374 109.347) (end 195.67652 112.04448) (width 0.254) (layer F.Cu) (net 3))
-  (segment (start 198.374 108.077) (end 198.374 109.347) (width 0.254) (layer F.Cu) (net 3))
-  (via (at 198.374 108.077) (size 0.889) (layers F.Cu B.Cu) (net 3))
-  (segment (start 198.374 99.441) (end 198.374 108.077) (width 0.254) (layer B.Cu) (net 3))
-  (segment (start 199.644 98.171) (end 198.374 99.441) (width 0.254) (layer B.Cu) (net 3))
+  (segment (start 193.294 112.04448) (end 194.91452 112.04448) (width 0.254) (layer F.Cu) (net 3) (status 400000))
+  (segment (start 198.374 99.06) (end 199.644 97.79) (width 0.254) (layer B.Cu) (net 3) (status 800000))
+  (segment (start 193.802 99.06) (end 198.374 99.06) (width 0.254) (layer B.Cu) (net 3))
+  (segment (start 193.294 99.568) (end 193.802 99.06) (width 0.254) (layer B.Cu) (net 3))
+  (segment (start 193.294 104.394) (end 193.294 99.568) (width 0.254) (layer B.Cu) (net 3))
+  (segment (start 193.929 105.029) (end 193.294 104.394) (width 0.254) (layer B.Cu) (net 3))
+  (segment (start 196.85 105.029) (end 193.929 105.029) (width 0.254) (layer B.Cu) (net 3))
+  (segment (start 198.247 106.426) (end 196.85 105.029) (width 0.254) (layer B.Cu) (net 3))
+  (segment (start 198.247 107.696) (end 198.247 106.426) (width 0.254) (layer B.Cu) (net 3))
+  (via (at 198.247 107.696) (size 0.889) (layers F.Cu B.Cu) (net 3))
+  (segment (start 198.247 108.712) (end 198.247 107.696) (width 0.254) (layer F.Cu) (net 3))
+  (segment (start 194.91452 112.04448) (end 198.247 108.712) (width 0.254) (layer F.Cu) (net 3))
   (segment (start 202.8952 108.8644) (end 205.1304 108.8644) (width 0.508) (layer F.Cu) (net 4))
   (segment (start 205.1304 108.8644) (end 205.486 109.22) (width 0.508) (layer F.Cu) (net 4))
@@
   (via (at 204.597 106.172) (size 0.889) (layers F.Cu B.Cu) (net 6))
   (segment (start 204.343 106.426) (end 204.597 106.172) (width 0.1524) (layer F.Cu) (net 6))
-  (segment (start 199.644 100.33) (end 202.184 102.87) (width 0.254) (layer F.Cu) (net 6))
-  (segment (start 202.184 105.7148) (end 202.8952 106.426) (width 0.254) (layer F.Cu) (net 6))
-  (segment (start 202.184 102.87) (end 202.184 105.7148) (width 0.254) (layer F.Cu) (net 6))
+  (segment (start 199.644 100.33) (end 202.184 102.743) (width 0.254) (layer F.Cu) (net 6) (status 400000))
+  (segment (start 202.2221 105.7529) (end 202.8952 106.426) (width 0.254) (layer F.Cu) (net 6) (status 800000))
+  (segment (start 202.184 102.743) (end 202.2221 105.7529) (width 0.254) (layer F.Cu) (net 6))
   (segment (start 198.12 123.19) (end 199.39 122.174) (width 0.254) (layer B.Cu) (net 7))
   (segment (start 200.914 107.569) (end 201.422 107.061) (width 0.254) (layer F.Cu) (net 7))
@@
   (segment (start 202.8952 107.2388) (end 202.7174 107.061) (width 0.254) (layer F.Cu) (net 7))
   (segment (start 198.374 99.06) (end 197.104 97.79) (width 0.254) (layer F.Cu) (net 7))
-  (segment (start 198.374 101.6) (end 198.374 99.06) (width 0.254) (layer F.Cu) (net 7))
-  (segment (start 198.755 101.981) (end 198.374 101.6) (width 0.254) (layer F.Cu) (net 7))
-  (segment (start 199.136 101.981) (end 198.755 101.981) (width 0.254) (layer F.Cu) (net 7))
-  (segment (start 200.533 101.981) (end 199.136 101.981) (width 0.254) (layer F.Cu) (net 7))
-  (segment (start 201.549 102.997) (end 200.533 101.981) (width 0.254) (layer F.Cu) (net 7))
-  (segment (start 201.549 105.791) (end 201.549 102.997) (width 0.254) (layer F.Cu) (net 7))
-  (segment (start 201.422 105.918) (end 201.549 105.791) (width 0.254) (layer F.Cu) (net 7))
+  (segment (start 198.374 100.838) (end 198.374 99.06) (width 0.254) (layer F.Cu) (net 7))
+  (segment (start 199.189788 101.537247) (end 198.374 100.838) (width 0.254) (layer F.Cu) (net 7))
+  (segment (start 200.025 101.473) (end 199.189788 101.537247) (width 0.254) (layer F.Cu) (net 7))
+  (segment (start 200.533 101.981) (end 200.025 101.473) (width 0.254) (layer F.Cu) (net 7))
+  (segment (start 201.676 102.997) (end 200.533 101.981) (width 0.254) (layer F.Cu) (net 7))
+  (segment (start 201.676 105.791) (end 201.676 102.997) (width 0.254) (layer F.Cu) (net 7))
+  (segment (start 201.422 105.918) (end 201.676 105.791) (width 0.254) (layer F.Cu) (net 7))
   (segment (start 201.422 107.061) (end 201.422 105.918) (width 0.254) (layer F.Cu) (net 7))
   (segment (start 202.7174 107.061) (end 201.422 107.061) (width 0.254) (layer F.Cu) (net 7))
@@
   (segment (start 200.8378 105.8418) (end 200.8378 106.6038) (width 0.254) (layer F.Cu) (net 10))
   (segment (start 200.914 105.7656) (end 200.8378 105.8418) (width 0.254) (layer F.Cu) (net 10))
-  (segment (start 197.104 100.33) (end 197.612 101.6) (width 0.254) (layer F.Cu) (net 10))
+  (segment (start 197.104 100.33) (end 198.374 101.6) (width 0.254) (layer F.Cu) (net 10) (status 400000))
   (segment (start 200.914 103.251) (end 200.914 104.4702) (width 0.254) (layer F.Cu) (net 10))
-  (segment (start 200.406 102.743) (end 200.914 103.251) (width 0.254) (layer F.Cu) (net 10))
-  (segment (start 198.628 102.616) (end 200.406 102.743) (width 0.254) (layer F.Cu) (net 10))
-  (segment (start 197.612 101.6) (end 198.628 102.616) (width 0.254) (layer F.Cu) (net 10))
+  (segment (start 199.891169 102.07121) (end 200.914 103.251) (width 0.254) (layer F.Cu) (net 10))
+  (segment (start 199.009199 102.07312) (end 199.891169 102.07121) (width 0.254) (layer F.Cu) (net 10))
+  (segment (start 198.374 101.6) (end 199.009199 102.07312) (width 0.254) (layer F.Cu) (net 10))
   (segment (start 182.499 108.458) (end 184.15 110.109) (width 0.508) (layer F.Cu) (net 11))
   (segment (start 191.89192 108.84408) (end 193.294 108.84408) (width 0.508) (layer F.Cu) (net 11))
@@
   (segment (start 206.248 108.204) (end 206.248 110.49) (width 0.254) (layer F.Cu) (net 16))
   (segment (start 209.042 106.553) (end 209.042 108.204) (width 0.508) (layer F.Cu) (net 16))
+  (segment (start 181.61 110.998) (end 182.499 111.887) (width 0.254) (layer F.Cu) (net 17))
+  (segment (start 181.102 107.188) (end 181.102 110.49) (width 0.254) (layer B.Cu) (net 17))
+  (segment (start 181.102 110.49) (end 181.61 110.998) (width 0.254) (layer B.Cu) (net 17))
+  (via (at 181.61 110.998) (size 0.889) (layers F.Cu B.Cu) (net 17))
+  (segment (start 182.88 105.41) (end 181.102 107.188) (width 0.254) (layer B.Cu) (net 17))
+  (via (at 186.055 113.792) (size 0.889) (layers F.Cu B.Cu) (net 17))
+  (segment (start 189.357 113.792) (end 186.055 113.792) (width 0.254) (layer F.Cu) (net 17))
+  (via (at 189.357 113.792) (size 0.889) (layers F.Cu B.Cu) (net 17))
+  (segment (start 189.357 111.887) (end 189.357 113.792) (width 0.254) (layer B.Cu) (net 17))
+  (via (at 189.357 111.887) (size 0.889) (layers F.Cu B.Cu) (net 17))
+  (segment (start 182.499 111.887) (end 189.357 111.887) (width 0.254) (layer F.Cu) (net 17))
   (segment (start 212.598 124.206) (end 212.598 119.888) (width 0.254) (layer F.Cu) (net 17))
   (segment (start 206.7306 121.1326) (end 207.518 121.92) (width 0.254) (layer F.Cu) (net 17))
@@
   (via (at 190.246 105.664) (size 0.889) (layers F.Cu B.Cu) (net 17))
   (segment (start 189.865 105.283) (end 190.246 105.664) (width 0.254) (layer F.Cu) (net 17))
-  (segment (start 182.88 105.41) (end 181.102 107.188) (width 0.254) (layer B.Cu) (net 17))
-  (via (at 181.61 110.998) (size 0.889) (layers F.Cu B.Cu) (net 17))
-  (segment (start 181.102 110.49) (end 181.61 110.998) (width 0.254) (layer B.Cu) (net 17))
-  (segment (start 181.102 107.188) (end 181.102 110.49) (width 0.254) (layer B.Cu) (net 17))
   (segment (start 196.89572 114.03584) (end 196.89572 115.77828) (width 0.254) (layer F.Cu) (net 17))
   (segment (start 196.89572 115.77828) (end 196.85 115.824) (width 0.254) (layer F.Cu) (net 17))
